File: hardware/Mainboard/Mainboard.kicad_sch (KiCad schematic)
At the start: 95 parts, among them CN1 NUCLE_F446RE_MORPHO_CN7, CN2 NUCLE_F446RE_MORPHO_CN10, J1 Conn_01x03_Pin, J10 Power, J12 Part_Cooling2, J13 Part_Cooling1, J2 Conn_01x03_Pin, J27 Conn_01x03_Pin, J28 Conn_01x02_Pin, J29 Conn_01x02_Pin, J30 Conn_01x02_Pin, J31 Conn_01x02_Pin, J32 Conn_01x02_Pin, J33 Conn_01x02_Pin, J34 Conn_01x02_Pin, J35 Conn_01x02_Pin, J36 Conn_01x04_Pin, J37 Conn_01x04_Pin, J38 Conn_01x02_Pin, J39 Conn_01x02_Pin, J4 Conn_01x02_Pin, J40 Conn_01x02_Pin, J41 Conn_01x02_Pin, J42 Conn_01x04_Pin, J43 Conn_01x04_Pin, J44 Conn_01x04_Pin, J45 Conn_01x02_Pin, J46 Conn_01x02_Pin, J47 Conn_01x02_Pin, J48 Conn_01x02_Pin, J49 Conn_01x04_Pin, J5 Conn_01x02_Pin, J50 Conn_01x04_Pin, J51 Conn_01x02_Pin, J52 Conn_01x02_Pin, J6 Hotend1, J8 Hotend2, J9 Bed, Q2 PSMN5R2-60YL, Q4 PSMN5R2-60YL, Q5 PSMN5R2-60YL, Q6 PSMN5R2-60YL, Q7 AO3400A, Q8 AO3400A, U1 MIC4426, U10 TMC2209_SILENTSTEPSTICK, U11 TMC2209_SILENTSTEPSTICK, U12 TMC2209_SILENTSTEPSTICK, U13 TMC2209_SILENTSTEPSTICK, U14 TMC2209_SILENTSTEPSTICK, U2 MIC4426, U8 TMC2209_SILENTSTEPSTICK, U9 TMC2209_SILENTSTEPSTICK

Commit message: Mainboard-3
Version 3 of Mainboard, (version 2 not uploaded)
Parts:
- removed C17, C18, C19, C20, C21, C22: 100µ, Capacitor_SMD:CP_Elec_8x10, symbol Device:C_Polarized
- removed C4, C5, C6, C7, C8, C9: 100n, Capacitor_SMD:C_0805_2012Metric, symbol Device:C
- removed J4, J5: Conn_01x02_Pin, symbol Connector:Conn_01x02_Pin
- added C14: 2.2uF (tantal), Capacitor_Tantalum_SMD:CP_EIA-3216-10_Kemet-I, symbol Device:C_Polarized
- added C15: 470pF, Capacitor_SMD:C_0805_2012Metric, symbol Device:C
- added C16, C17, C18, C19, C20, C21, C22: 100n, Capacitor_SMD:C_0805_2012Metric, symbol Device:C
- added C24, C25, C36, C37, C38, C39, C40: 100µ, Capacitor_SMD:CP_Elec_8x10, symbol Device:C_Polarized
- added C26, C33, C34, C35: 2.2uF, Capacitor_SMD:C_0805_2012Metric, symbol Device:C
- added C27: 0.1uF, Capacitor_SMD:C_0805_2012Metric, symbol Device:C
- added C28: 4.7pF, Capacitor_SMD:C_0805_2012Metric, symbol Device:C
- added C29: 4.7nF, Capacitor_SMD:C_0805_2012Metric, symbol Device:C
- added C30, C31, C32: 47uF, Capacitor_SMD:C_0805_2012Metric, symbol Device:C
- added D1: B560C, Diode_SMD:D_SMC, symbol Device:D
- added H1, H2, H3, H4: MountingHole, MountingHole:MountingHole_2.7mm_M2.5_Pad_Via, symbol Mechanical:MountingHole
- added J53: R_MS2, Connector_PinHeader_2.54mm:PinHeader_1x02_P2.54mm_Vertical, symbol Connector:Conn_01x02_Pin
- added J54: R_MS1, Connector_PinHeader_2.54mm:PinHeader_1x02_P2.54mm_Vertical, symbol Connector:Conn_01x02_Pin
- added J55: R_Motor, Connector_PinHeader_2.54mm:PinHeader_1x04_P2.54mm_Vertical, symbol Connector:Conn_01x04_Pin
- added L1: 7.2uH, Inductor_SMD:L_Wuerth_WE-PDF, symbol Device:L
- added R13: 16.9k, Resistor_SMD:R_0805_2012Metric, symbol Device:R
- added R14: 442k, Resistor_SMD:R_0805_2012Metric, symbol Device:R
- added R19: 90.9k, Resistor_SMD:R_0805_2012Metric, symbol Device:R
- added R20: 243k, Resistor_SMD:R_0805_2012Metric, symbol Device:R
- added R21: 53.6k, Resistor_SMD:R_0805_2012Metric, symbol Device:R
- added R22: 10.2k, Resistor_SMD:R_0805_2012Metric, symbol Device:R
- added R23, R24: 1k, Resistor_SMD:R_0805_2012Metric, symbol Device:R_Small
- added R25: 11k, Resistor_SMD:R_0805_2012Metric, symbol Device:R
- added R26: 100k, Resistor_SMD:R_0805_2012Metric, symbol Device:R
- added U15: R, FlexPrint:MODULE_TMC2209_SILENTSTEPSTICK, symbol FlexPrint:TMC2209_SILENTSTEPSTICK
- added U3: TPS54560BDDA, Package_SO:Texas_R-PDSO-G8_EP2.95x4.9mm_Mask2.4x3.1mm_ThermalVias, symbol Regulator_Switching:TPS54560BDDA
- added U4: MIC5219-3.3YM5, Package_TO_SOT_SMD:SOT-23-5, symbol Regulator_Linear:MIC5219-3.3YM5
- F1, F2, F3, F4: footprint (none) -> Fuse:Fuse_1206_3216Metric
- J1: value Conn_01x03_Pin -> X_END; footprint (none) -> Connector_JST:JST_XH_B3B-XH-A_1x03_P2.50mm_Vertical
- J10, J6, J8, J9: footprint (none) -> TerminalBlock:TerminalBlock_bornier-2_P5.08mm
- J12, J13: footprint (none) -> Connector_JST:JST_XH_B2B-XH-A_1x02_P2.50mm_Vertical
- J2: value Conn_01x03_Pin -> Y_END; footprint (none) -> Connector_JST:JST_XH_B3B-XH-A_1x03_P2.50mm_Vertical
- J27: value Conn_01x03_Pin -> Z_END; footprint (none) -> Connector_JST:JST_XH_B3B-XH-A_1x03_P2.50mm_Vertical
- J28: value Conn_01x02_Pin -> X_MS2; footprint (none) -> Connector_PinHeader_2.54mm:PinHeader_1x02_P2.54mm_Vertical
- J29: value Conn_01x02_Pin -> HE1_therm; footprint (none) -> Connector_JST:JST_XH_B2B-XH-A_1x02_P2.50mm_Vertical
- J3: value ~ -> +12V; footprint (none) -> TerminalBlock:TerminalBlock_bornier-2_P5.08mm
- J30: value Conn_01x02_Pin -> Bed_therm; footprint (none) -> Connector_JST:JST_XH_B2B-XH-A_1x02_P2.50mm_Vertical
- J31: value Conn_01x02_Pin -> Z1_MS2; footprint (none) -> Connector_PinHeader_2.54mm:PinHeader_1x02_P2.54mm_Vertical
- J32: value Conn_01x02_Pin -> X_MS1; footprint (none) -> Connector_PinHeader_2.54mm:PinHeader_1x02_P2.54mm_Vertical
- J33: value Conn_01x02_Pin -> Z1_MS1; footprint (none) -> Connector_PinHeader_2.54mm:PinHeader_1x02_P2.54mm_Vertical
- J34: value Conn_01x02_Pin -> Z4_MS2; footprint (none) -> Connector_PinHeader_2.54mm:PinHeader_1x02_P2.54mm_Vertical
- J35: value Conn_01x02_Pin -> Z4_MS1; footprint (none) -> Connector_PinHeader_2.54mm:PinHeader_1x02_P2.54mm_Vertical
- J36: value Conn_01x04_Pin -> X_Motor; footprint (none) -> Connector_PinHeader_2.54mm:PinHeader_1x04_P2.54mm_Vertical
- J37: value Conn_01x04_Pin -> Z1_Motor; footprint (none) -> Connector_PinHeader_2.54mm:PinHeader_1x04_P2.54mm_Vertical
- J38: value Conn_01x02_Pin -> Y_MS2; footprint (none) -> Connector_PinHeader_2.54mm:PinHeader_1x02_P2.54mm_Vertical
- J39: value Conn_01x02_Pin -> Z2_MS2; footprint (none) -> Connector_PinHeader_2.54mm:PinHeader_1x02_P2.54mm_Vertical
- J40: value Conn_01x02_Pin -> Y_MS1; footprint (none) -> Connector_PinHeader_2.54mm:PinHeader_1x02_P2.54mm_Vertical
- J41: value Conn_01x02_Pin -> Z2_MS1; footprint (none) -> Connector_PinHeader_2.54mm:PinHeader_1x02_P2.54mm_Vertical
- J42: value Conn_01x04_Pin -> Z4_Motor; footprint (none) -> Connector_PinHeader_2.54mm:PinHeader_1x04_P2.54mm_Vertical
- J43: value Conn_01x04_Pin -> Y_Motor; footprint (none) -> Connector_PinHeader_2.54mm:PinHeader_1x04_P2.54mm_Vertical
- J44: value Conn_01x04_Pin -> Z2_Motor; footprint (none) -> Connector_PinHeader_2.54mm:PinHeader_1x04_P2.54mm_Vertical
- J45: value Conn_01x02_Pin -> E_MS2; footprint (none) -> Connector_PinHeader_2.54mm:PinHeader_1x02_P2.54mm_Vertical
- J46: value Conn_01x02_Pin -> Z3_MS2; footprint (none) -> Connector_PinHeader_2.54mm:PinHeader_1x02_P2.54mm_Vertical
- J47: value Conn_01x02_Pin -> E_MS1; footprint (none) -> Connector_PinHeader_2.54mm:PinHeader_1x02_P2.54mm_Vertical
- J48: value Conn_01x02_Pin -> Z3_MS1; footprint (none) -> Connector_PinHeader_2.54mm:PinHeader_1x02_P2.54mm_Vertical
- J49: value Conn_01x04_Pin -> E_Motor; footprint (none) -> Connector_PinHeader_2.54mm:PinHeader_1x04_P2.54mm_Vertical
- J50: value Conn_01x04_Pin -> Z3_Motor; footprint (none) -> Connector_PinHeader_2.54mm:PinHeader_1x04_P2.54mm_Vertical
- J51: value Conn_01x02_Pin -> PWR_therm; footprint (none) -> Connector_JST:JST_XH_B2B-XH-A_1x02_P2.50mm_Vertical
- J52: value Conn_01x02_Pin -> HE2_therm; footprint (none) -> Connector_JST:JST_XH_B2B-XH-A_1x02_P2.50mm_Vertical
- J7: value ~ -> +24V; footprint (none) -> TerminalBlock:TerminalBlock_bornier-2_P5.08mm
- U1, U2: footprint (none) -> Package_SO:SOIC-8_3.9x4.9mm_P1.27mm
- U10: value TMC2209_SILENTSTEPSTICK -> Z4; symbol PacFab:TMC2209_SILENTSTEPSTICK -> FlexPrint:TMC2209_SILENTSTEPSTICK; Availability (none) -> In Stock; Check_prices (none) -> https://www.snapeda.com/parts/TMC2209%20SILENTSTEPSTICK/Tri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; Description_1 (none) -> TMC2209 Motor Controller/Driver Power Management Evaluation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; MANUFACTURER (none) -> Trinamic Motion Control GmbH; MF (none) -> Trinamic Motion Control GmbH; MP (none) -> TMC2209 SILENTSTEPSTICK; PARTREV (none) -> 1.20; Package (none) -> None; Price (none) -> None; SNAPEDA_PN (none) -> TMC2209 SILENTSTEPSTICK; STANDARD (none) -> Manufacturer Recommendations; SnapEDA_Link (none) -> https://www.snapeda.com/parts/TMC2209%20SILENTSTEPSTICK/Tri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
- U11: value TMC2209_SILENTSTEPSTICK -> Y; footprint (none) -> FlexPrint:MODULE_TMC2209_SILENTSTEPSTICK; symbol PacFab:TMC2209_SILENTSTEPSTICK -> FlexPrint:TMC2209_SILENTSTEPSTICK; Availability (none) -> In Stock; Check_prices (none) -> https://www.snapeda.com/parts/TMC2209%20SILENTSTEPSTICK/Tri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; Description_1 (none) -> TMC2209 Motor Controller/Driver Power Management Evaluation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; MANUFACTURER (none) -> Trinamic Motion Control GmbH; MF (none) -> Trinamic Motion Control GmbH; MP (none) -> TMC2209 SILENTSTEPSTICK; PARTREV (none) -> 1.20; Package (none) -> None; Price (none) -> None; SNAPEDA_PN (none) -> TMC2209 SILENTSTEPSTICK; STANDARD (none) -> Manufacturer Recommendations; SnapEDA_Link (none) -> https://www.snapeda.com/parts/TMC2209%20SILENTSTEPSTICK/Tri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
- U12: value TMC2209_SILENTSTEPSTICK -> Z2; footprint (none) -> FlexPrint:MODULE_TMC2209_SILENTSTEPSTICK; symbol PacFab:TMC2209_SILENTSTEPSTICK -> FlexPrint:TMC2209_SILENTSTEPSTICK; Availability (none) -> In Stock; Check_prices (none) -> https://www.snapeda.com/parts/TMC2209%20SILENTSTEPSTICK/Tri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; Description_1 (none) -> TMC2209 Motor Controller/Driver Power Management Evaluation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; MANUFACTURER (none) -> Trinamic Motion Control GmbH; MF (none) -> Trinamic Motion Control GmbH; MP (none) -> TMC2209 SILENTSTEPSTICK; PARTREV (none) -> 1.20; Package (none) -> None; Price (none) -> None; SNAPEDA_PN (none) -> TMC2209 SILENTSTEPSTICK; STANDARD (none) -> Manufacturer Recommendations; SnapEDA_Link (none) -> https://www.snapeda.com/parts/TMC2209%20SILENTSTEPSTICK/Tri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
- U13: value TMC2209_SILENTSTEPSTICK -> E; footprint (none) -> FlexPrint:MODULE_TMC2209_SILENTSTEPSTICK; symbol PacFab:TMC2209_SILENTSTEPSTICK -> FlexPrint:TMC2209_SILENTSTEPSTICK; Availability (none) -> In Stock; Check_prices (none) -> https://www.snapeda.com/parts/TMC2209%20SILENTSTEPSTICK/Tri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; Description_1 (none) -> TMC2209 Motor Controller/Driver Power Management Evaluation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; MANUFACTURER (none) -> Trinamic Motion Control GmbH; MF (none) -> Trinamic Motion Control GmbH; MP (none) -> TMC2209 SILENTSTEPSTICK; PARTREV (none) -> 1.20; Package (none) -> None; Price (none) -> None; SNAPEDA_PN (none) -> TMC2209 SILENTSTEPSTICK; STANDARD (none) -> Manufacturer Recommendations; SnapEDA_Link (none) -> https://www.snapeda.com/parts/TMC2209%20SILENTSTEPSTICK/Tri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
- U14: value TMC2209_SILENTSTEPSTICK -> Z3; footprint (none) -> FlexPrint:MODULE_TMC2209_SILENTSTEPSTICK; symbol PacFab:TMC2209_SILENTSTEPSTICK -> FlexPrint:TMC2209_SILENTSTEPSTICK; Availability (none) -> In Stock; Check_prices (none) -> https://www.snapeda.com/parts/TMC2209%20SILENTSTEPSTICK/Tri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; Description_1 (none) -> TMC2209 Motor Controller/Driver Power Management Evaluation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; MANUFACTURER (none) -> Trinamic Motion Control GmbH; MF (none) -> Trinamic Motion Control GmbH; MP (none) -> TMC2209 SILENTSTEPSTICK; PARTREV (none) -> 1.20; Package (none) -> None; Price (none) -> None; SNAPEDA_PN (none) -> TMC2209 SILENTSTEPSTICK; STANDARD (none) -> Manufacturer Recommendations; SnapEDA_Link (none) -> https://www.snapeda.com/parts/TMC2209%20SILENTSTEPSTICK/Tri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
- U8: value TMC2209_SILENTSTEPSTICK -> X; footprint (none) -> FlexPrint:MODULE_TMC2209_SILENTSTEPSTICK; symbol PacFab:TMC2209_SILENTSTEPSTICK -> FlexPrint:TMC2209_SILENTSTEPSTICK; Availability (none) -> In Stock; Check_prices (none) -> https://www.snapeda.com/parts/TMC2209%20SILENTSTEPSTICK/Tri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; Description_1 (none) -> TMC2209 Motor Controller/Driver Power Management Evaluation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; MANUFACTURER (none) -> Trinamic Motion Control GmbH; MF (none) -> Trinamic Motion Control GmbH; MP (none) -> TMC2209 SILENTSTEPSTICK; PARTREV (none) -> 1.20; Package (none) -> None; Price (none) -> None; SNAPEDA_PN (none) -> TMC2209 SILENTSTEPSTICK; STANDARD (none) -> Manufacturer Recommendations; SnapEDA_Link (none) -> https://www.snapeda.com/parts/TMC2209%20SILENTSTEPSTICK/Tri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
- U9: value TMC2209_SILENTSTEPSTICK -> Z1; footprint (none) -> FlexPrint:MODULE_TMC2209_SILENTSTEPSTICK; symbol PacFab:TMC2209_SILENTSTEPSTICK -> FlexPrint:TMC2209_SILENTSTEPSTICK; Availability (none) -> In Stock; Check_prices (none) -> https://www.snapeda.com/parts/TMC2209%20SILENTSTEPSTICK/Tri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; Description_1 (none) -> TMC2209 Motor Controller/Driver Power Management Evaluation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; MANUFACTURER (none) -> Trinamic Motion Control GmbH; MF (none) -> Trinamic Motion Control GmbH; MP (none) -> TMC2209 SILENTSTEPSTICK; PARTREV (none) -> 1.20; Package (none) -> None; Price (none) -> None; SNAPEDA_PN (none) -> TMC2209 SILENTSTEPSTICK; STANDARD (none) -> Manufacturer Recommendations; SnapEDA_Link (none) -> https://www.snapeda.com/parts/TMC2209%20SILENTSTEPSTICK/Tri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
Connections:
- net VCC is gone; now on net +3V3: J28.1 (Pin_1), J31.1 (Pin_1), J32.1 (Pin_1), J33.1 (Pin_1), J34.1 (Pin_1), J35.1 (Pin_1), J38.1 (Pin_1), J39.1 (Pin_1), J40.1 (Pin_1), J41.1 (Pin_1), J45.1 (Pin_1), J46.1 (Pin_1), J47.1 (Pin_1), J48.1 (Pin_1)
- net +12V: now also U1.6 (V+), U2.6 (V+), C26.1, C33.1, C34.1, C35.1, R14.1, U3.2 (VIN); no longer C23.1
- net +24V: now also C23.1, U10.8 (VM), U11.8 (VM), U12.8 (VM), U13.8 (VM), U14.8 (VM), U8.8 (VM), U9.8 (VM), C24.1, C25.1, C36.1, C37.1, C38.1, C39.1, C40.1, R26.1, U15.8 (VM)
- net +3V3: now also U10.2 (VIO), U11.2 (VIO), U12.2 (VIO), U13.2 (VIO), U14.2 (VIO), U8.2 (VIO), U9.2 (VIO), C14.1, C16.1, C17.1, C18.1, C19.1, C20.1, C21.1, C22.1, J53.1 (Pin_1), J54.1 (Pin_1), U15.2 (VIO), U4.5 (OUT)
- net +5V: now also C30.1, C31.1, C32.1, L1.2, R21.1, U4.1 (IN), U4.3 (EN)
- net E_1A: now also U13.3 (M1A); no longer U13.4 (M1A)
- net E_1B: now also U13.5 (M1B); no longer U13.3 (M1B)
- net E_2A: now also U13.4 (M2A); no longer U13.5 (M2A)
- net GND: now also C10.2, C23.2, U1.3 (GND), U2.3 (GND), C14.2, C15.2, C16.2, C17.2, C18.2, C19.2, C20.2, C21.2, C22.2, C24.2, C25.2, C26.2, C28.2, C29.2, C30.2, C31.2, C32.2, C33.2, C34.2, C35.2, C36.2, C37.2, C38.2, C39.2, C40.2, D1.2 (A), R19.2, R20.2, R22.2, R25.2, U15.1 (GND), U15.7 (GND), U3.7 (GND), U3.9 (GND), U4.2 (GND)
- net PCF1: now also CN2.17 (Pin_17); no longer CN1.30 (Pin_30)
- net PCF2: now also CN1.21 (Pin_21); no longer CN1.28 (Pin_28)
- net X_1A: now also U8.3 (M1A); no longer U8.4 (M1A)
- net X_1B: now also U8.5 (M1B); no longer U8.3 (M1B)
- net X_2A: now also U8.4 (M2A); no longer U8.5 (M2A)
- net X_END: now also CN1.25 (Pin_25); no longer CN1.23 (Pin_23)
- net Y_1A: now also U11.3 (M1A); no longer U11.4 (M1A)
- net Y_1B: now also U11.5 (M1B); no longer U11.3 (M1B)
- net Y_2A: now also U11.4 (M2A); no longer U11.5 (M2A)
- net Y_DIR: now also CN1.1 (Pin_1); no longer CN2.16 (Pin_16)
- net Y_EN: now also CN1.2 (Pin_2); no longer CN2.12 (Pin_12)
- net Y_END: now also CN1.23 (Pin_23); no longer CN1.25 (Pin_25)
- net Y_STEP: now also CN1.4 (Pin_4); no longer CN2.14 (Pin_14)
- net Z1_1A: now also U9.3 (M1A); no longer U9.4 (M1A)
- net Z1_1B: now also U9.5 (M1B); no longer U9.3 (M1B)
- net Z1_2A: now also U9.4 (M2A); no longer U9.5 (M2A)
- net Z1_STEP: now also CN2.23 (Pin_23); no longer CN2.17 (Pin_17)
- net Z2_1A: now also U12.3 (M1A); no longer U12.4 (M1A)
- net Z2_1B: now also U12.5 (M1B); no longer U12.3 (M1B)
- net Z2_2A: now also U12.4 (M2A); no longer U12.5 (M2A)
- net Z2_DIR: now also CN1.17 (Pin_17); no longer CN2.25 (Pin_25)
- net Z2_EN: now also CN1.13 (Pin_13); no longer CN2.21 (Pin_21)
- net Z2_STEP: now also CN1.15 (Pin_15); no longer CN2.23 (Pin_23)
- net Z3_1A: now also U14.3 (M1A); no longer U14.4 (M1A)
- net Z3_1B: now also U14.5 (M1B); no longer U14.3 (M1B)
- net Z3_2A: now also U14.4 (M2A); no longer U14.5 (M2A)
- net Z3_DIR: now also CN2.29 (Pin_29); no longer CN2.31 (Pin_31)
- net Z3_EN: now also CN2.25 (Pin_25); no longer CN2.27 (Pin_27)
- net Z3_STEP: now also CN2.27 (Pin_27); no longer CN2.29 (Pin_29)
- net Z4_1A: now also U10.3 (M1A); no longer U10.4 (M1A)
- net Z4_1B: now also U10.5 (M1B); no longer U10.3 (M1B)
- net Z4_2A: now also U10.4 (M2A); no longer U10.5 (M2A)
- net Z4_DIR: now also CN2.4 (Pin_4); no longer CN2.37 (Pin_37)
- net Z4_EN: now also CN2.31 (Pin_31); no longer CN2.33 (Pin_33)
- net Z4_STEP: now also CN2.2 (Pin_2); no longer CN2.35 (Pin_35)
- removed net M_DIAG: U10.18 (DIAG), U11.18 (DIAG), U12.18 (DIAG), U13.18 (DIAG), U14.18 (DIAG), U8.18 (DIAG), U9.18 (DIAG)
- net M_UART renamed uart2_tmc
- net uart2_tmc: now also CN1.28 (Pin_28), R23.2; no longer U11.12 (UART), U13.12 (UART), U8.12 (UART)
- new net: J53.2 (Pin_2), U15.14 (MS2)
- new net: R25.1, R26.2, U3.3 (EN)
- new net: C27.1, D1.1 (K), L1.1, U3.1 (BOOT)
- new net: R20.1, U3.4 (RT/CLK)
- new net: CN2.33 (Pin_33), R24.2
- new net: J54.2 (Pin_2), U15.15 (MS1)
- new net: C29.1, R13.2
- new net: R14.2, R19.1
- new net: CN1.30 (Pin_30), R23.1
- new net: C28.1, R13.1, U3.6 (COMP)
- new net: C27.2, U3.8 (SW)
- new net: C15.1, U4.4 (BP)
- new net FB: R21.2, R22.1, U3.5 (FB)
- new net R_1A: J55.4 (Pin_4), U15.3 (M1A)
- new net R_1B: J55.2 (Pin_2), U15.5 (M1B)
- new net R_2A: J55.3 (Pin_3), U15.4 (M2A)
- new net R_2B: J55.1 (Pin_1), U15.6 (M2B)
- new net R_DIR: CN2.16 (Pin_16), U15.9 (DIR)
- new net R_EN: CN2.12 (Pin_12), U15.16 (~{EN})
- new net R_STEP: CN2.14 (Pin_14), U15.10 (STEP)
- new net uart1_tmc: CN2.21 (Pin_21), R24.1, U11.12 (UART), U13.12 (UART), U15.12 (UART), U8.12 (UART)
- no-connect marks 40 -> 49
Other:
- note added: "4 Treiber pro Uart, da nur 4 Adressen einstellbar"
- note added: "4 Z-Achsen, 1 X-Achse, 1 Y-Achse, 1 Extruder und 1 Reserve Treiber"
- note added: "5V and 3.3V Supply"
- note added: "Reserve motor"
- note added: "x nicht direkt am Pin = ADC Pin"
- note removed: "Buck 12V to 3.3V"
- company: (none) -> Flexprint
- title: (none) -> Mainboard
- moved on the sheet: C1, C11, CN1, CN2, J1, J2, J27, J28, J3, J31, J32, J33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

Commit message: mainboard v2
Changed lines of the file:
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@@
+		)
+	)
+	(text_box "TODO:\n	-part cooling fans auf 24V\n	-mehr versorgunsanschlüsse (5V,12V usw)\n	-Verpolschutz\n\nEventuelle TODO's:\n	-wenn viel mehr funktionen benötigt werden -> eigenen µC 	verwenden statt devBoard\n		-beschaltung dafür	\n		-USB für Raspi"
+		(exclude_from_sim no)
+		(at 422.91 12.7 0)
+		(size 73.66 44.45)
+		(margins 0.9525 0.9525 0.9525 0.9525)
+		(stroke
+			(width 0)
+			(type solid)
+		)
+		(fill
+			(type none)
+		)
+		(effects
+			(font
+				(size 1.27 1.27)
+			)
+			(justify left top)
 		)
 	)

Commit message: graphics/logo
Other:
- note added: "3 Z-Achsen, 1 X-Achse, 1 Y-Achse, 2 Extruder und 1 Reserve Treiber"
- note added: "E2 motor"
- note removed: "4 Z-Achsen, 1 X-Achse, 1 Y-Achse, 1 Extruder und 1 Reserve Treiber"
- note removed: "Z4 motor"
Changed lines of the file:
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@@
 		)
 	)
-	(text "Z4 motor"
+	(text "E2 motor"
 		(exclude_from_sim no)
 		(at 256.286 167.386 0)
@@
 		)
 	)
-	(text "4 Z-Achsen, 1 X-Achse, 1 Y-Achse, 1 Extruder und 1 Reserve Treiber"
+	(text "3 Z-Achsen, 1 X-Achse, 1 Y-Achse, 2 Extruder und 1 Reserve Treiber"
 		(exclude_from_sim no)
 		(at 320.802 110.744 0)
@@
 		)
 	)
-	(text_box "TODO:\n	-part cooling fans auf 24V\n	-mehr versorgunsanschlüsse (5V,12V usw)\n	-Verpolschutz\n\nEventuelle TODO's:\n	-wenn viel mehr funktionen benötigt werden -> eigenen µC 	verwenden statt devBoard\n		-beschaltung dafür	\n		-USB für Raspi"
+	(text_box "TODO:\n	-part cooling fans auf 24V (derzeitige Treiber halten 24V auch aus)\n	-mehr versorgunsanschlüsse (5V,12V usw)\n	-Verpolschutz\n	-Position Nucleo auf der Platine ändern!!!\n\nEventuelle TODO's:\n	-wenn viel mehr funktionen benötigt werden -> eigenen µC verwenden statt devBoard\n		-beschaltung dafür	\n		-USB für Raspi"
 		(exclude_from_sim no)
-		(at 422.91 12.7 0)
-		(size 73.66 44.45)
+		(at 422.91 10.16 0)
+		(size 105.41 44.45)
 		(margins 0.9525 0.9525 0.9525 0.9525)
 		(stroke
@@
 	(wire
 		(pts
+			(xy 359.41 224.79) (xy 361.95 224.79)
+		)
+		(stroke
+			(width 0)
+			(type default)
+		)
+	)
+	(wire
+		(pts
 			(xy 236.22 265.43) (xy 234.95 265.43)
 		)
@@
 	(wire
 		(pts
-			(xy 320.04 179.07) (xy 322.58 179.07)
+			(xy 321.31 179.07) (xy 322.58 179.07)
 		)
 		(stroke
@@
 	(symbol
 		(lib_id "power:+5V")
-		(at 361.95 224.79 0)
+		(at 359.41 224.79 0)
 		(unit 1)
 		(exclude_from_sim no)
@@
 		(fields_autoplaced yes)
 		(property "Reference" "#PWR030"
-			(at 361.95 228.6 0)
+			(at 359.41 228.6 0)
 			(effects
 				(font
@@
 		)
 		(property "Value" "+5V"
-			(at 361.95 219.71 0)
+			(at 359.41 219.71 0)
 			(effects
 				(font
@@
 		)
 		(property "Footprint" ""
-			(at 361.95 224.79 0)
+			(at 359.41 224.79 0)
 			(effects
 				(font
@@
 		)
 		(property "Datasheet" ""
-			(at 361.95 224.79 0)
+			(at 359.41 224.79 0)
 			(effects
 				(font
@@
 		)
 		(property "Description" "Power symbol creates a global label with name \"+5V\""
-			(at 361.95 224.79 0)
+			(at 359.41 224.79 0)
 			(effects
 				(font
@@
 	(symbol
 		(lib_id "power:GND")
-		(at 320.04 179.07 0)
+		(at 321.31 179.07 270)
 		(unit 1)
 		(exclude_from_sim no)
@@
 		(fields_autoplaced yes)
 		(property "Reference" "#PWR0126"
-			(at 320.04 185.42 0)
+			(at 314.96 179.07 0)
 			(effects
 				(font
@@
 		)
 		(property "Value" "GND"
-			(at 320.04 184.15 0)
+			(at 320.04 175.26 90)
 			(effects
 				(font
@@
 		)
 		(property "Footprint" ""
-			(at 320.04 179.07 0)
+			(at 321.31 179.07 0)
 			(effects
 				(font
@@
 		)
 		(property "Datasheet" ""
-			(at 320.04 179.07 0)
+			(at 321.31 179.07 0)
 			(effects
 				(font
@@
 		)
 		(property "Description" "Power symbol creates a global label with name \"GND\" , ground"
-			(at 320.04 179.07 0)
+			(at 321.31 179.07 0)
 			(effects
 				(font
