File: hardware/Mainboard/Mainboard.kicad_sch (KiCad schematic)
At the start: 129 parts, among them CN1 NUCLE_F446RE_MORPHO_CN7, CN2 NUCLE_F446RE_MORPHO_CN10, J1 X_END, J10 Power, J12 Part_Cooling2, J13 Part_Cooling1, J2 Y_END, J27 Z_END, J28 X_MS2, J29 HE1_therm, J3 +12V, J30 Bed_therm, J31 Z1_MS2, J32 X_MS1, J33 Z1_MS1, J34 Z4_MS2, J35 Z4_MS1, J36 X_Motor, J37 Z1_Motor, J38 Y_MS2, J39 Z2_MS2, J40 Y_MS1, J41 Z2_MS1, J42 Z4_Motor, J43 Y_Motor, J44 Z2_Motor, J45 E_MS2, J46 Z3_MS2, J47 E_MS1, J48 Z3_MS1, J49 E_Motor, J50 Z3_Motor, J51 PWR_therm, J52 HE2_therm, J53 R_MS2, J54 R_MS1, J55 R_Motor, J6 Hotend1, J7 +24V, J8 Hotend2, J9 Bed, Q2 PSMN5R2-60YL, Q4 PSMN5R2-60YL, Q5 PSMN5R2-60YL, Q6 PSMN5R2-60YL, Q7 AO3400A, Q8 AO3400A, U1 MIC4426, U10 Z4, U11 Y, U12 Z2, U13 E, U14 Z3, U15 R, U2 MIC4426, U3 TPS54560BDDA, U4 MIC5219-3.3YM5, U8 X, U9 Z1

Commit message: finalization of the project
the project is officially finished and running.
there will be further development when theres time to spare,
Connections:
- net Z4_1A renamed E2_1A
- net Z4_1B renamed E2_1B
- net Z4_2A renamed E2_2A
- net Z4_2B renamed E2_2B
- net Z4_DIR renamed E2_DIR
- net Z4_EN renamed E2_EN
- net Z4_STEP renamed E2_STEP
Changed lines of the file:
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@@
 		)
 	)
-	(text_box "TODO:\n	-part cooling fans auf 24V (derzeitige Treiber halten 24V auch aus)\n	-mehr versorgunsanschlüsse (5V,12V usw)\n	-Verpolschutz\n	-Position Nucleo auf der Platine ändern!!!\n\nEventuelle TODO's:\n	-wenn viel mehr funktionen benötigt werden -> eigenen µC verwenden statt devBoard\n		-beschaltung dafür	\n		-USB für Raspi"
+	(text_box "TODO:\n	-part cooling fans auf 24V (derzeitige Treiber halten 24V auch aus)\n	-mehr versorgunsanschlüsse (5V,12V usw)\n	-Verpolschutz\n	-Position Nucleo auf der Platine ändern!!!\n\nEventuelle TODO's:\n	-wenn viel mehr funktionen benötigt werden -> eigenen µC verwenden statt devBoard\n		-beschaltung dafür	\n		-USB für Raspi\n\nWICHTIG:\n	-MIC FET-Treiber ERSETZT DURCH ADP3634!!"
 		(exclude_from_sim no)
 		(at 422.91 10.16 0)
@@
 		)
 	)
-	(label "Z4_2B"
+	(label "E2_2B"
 		(at 274.32 201.93 0)
 		(effects
@@
 		)
 	)
-	(label "Z4_1B"
+	(label "E2_1B"
 		(at 274.32 199.39 0)
 		(effects
@@
 		)
 	)
-	(label "Z4_1A"
+	(label "E2_1A"
 		(at 274.32 194.31 0)
 		(effects
@@
 		)
 	)
-	(label "Z4_2A"
+	(label "E2_2A"
 		(at 274.32 196.85 0)
 		(effects
@@
 		)
 	)
-	(global_label "Z4_STEP"
+	(global_label "E2_STEP"
 		(shape input)
 		(at 238.76 191.77 180)
@@
 		)
 		(property "Intersheetrefs" "${INTERSHEET_REFS}"
-			(at 227.7921 191.77 0)
+			(at 228.5068 191.77 0)
 			(effects
 				(font
@@
 		)
 	)
-	(global_label "Z4_EN"
+	(global_label "E2_EN"
 		(shape output)
 		(at 226.06 142.24 180)
@@
 		)
 		(property "Intersheetrefs" "${INTERSHEET_REFS}"
-			(at 217.2087 142.24 0)
+			(at 217.9234 142.24 0)
 			(effects
 				(font
@@
 		)
 	)
-	(global_label "Z4_DIR"
+	(global_label "E2_DIR"
 		(shape output)
 		(at 252.73 106.68 0)
@@
 		)
 		(property "Intersheetrefs" "${INTERSHEET_REFS}"
-			(at 261.5924 106.68 0)
+			(at 261.5319 106.68 0)
 			(effects
 				(font
@@
 		)
 	)
-	(global_label "Z4_EN"
+	(global_label "E2_EN"
 		(shape input)
 		(at 238.76 186.69 180)
@@
 		)
 		(property "Intersheetrefs" "${INTERSHEET_REFS}"
-			(at 229.9087 186.69 0)
+			(at 230.6234 186.69 0)
 			(effects
 				(font
@@
 		)
 	)
-	(global_label "Z4_STEP"
+	(global_label "E2_STEP"
 		(shape output)
 		(at 252.73 104.14 0)
@@
 		)
 		(property "Intersheetrefs" "${INTERSHEET_REFS}"
-			(at 263.0437 104.14 0)
+			(at 262.9832 104.14 0)
 			(effects
 				(font
@@
 		)
 	)
-	(global_label "Z4_DIR"
+	(global_label "E2_DIR"
 		(shape input)
 		(at 238.76 194.31 180)
@@
 		)
 		(property "Intersheetrefs" "${INTERSHEET_REFS}"
-			(at 229.2434 194.31 0)
+			(at 229.9581 194.31 0)
 			(effects
 				(font
