File: hardware/TMC2209_driver/TMC2209_driver/TMC2209_driver.kicad_sch (KiCad schematic)
At the start: 20 parts, among them J1 Conn_01x08, J2 Conn_01x08, J3 Conn_01x02

Commit message: finalization of the project
the project is officially finished and running.
there will be further development when theres time to spare,
Other:
- company: (none) -> FlexPrint
- title: (none) -> Treiberplatine
- moved on the sheet: C6, C7
Changed lines of the file:
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@@
 	(generator_version "9.0")
 	(paper "A4")
+	(title_block
+		(title "Treiberplatine")
+		(date "2026-01-12")
+		(rev "3")
+		(company "FlexPrint")
+	)
 	(junction
 		(at 137.16 125.73)
@@
 	)
 	(junction
-		(at 124.46 62.23)
+		(at 128.27 62.23)
 		(diameter 0)
 		(color 0 0 0 0)
@@
 	)
 	(junction
-		(at 124.46 50.8)
+		(at 128.27 50.8)
 		(diameter 0)
 		(color 0 0 0 0)
@@
 	)
 	(junction
-		(at 124.46 58.42)
+		(at 128.27 58.42)
 		(diameter 0)
 		(color 0 0 0 0)
@@
 	(wire
 		(pts
-			(xy 115.57 58.42) (xy 124.46 58.42)
+			(xy 119.38 58.42) (xy 128.27 58.42)
 		)
 		(stroke
@@
 	(wire
 		(pts
-			(xy 124.46 62.23) (xy 124.46 58.42)
+			(xy 128.27 62.23) (xy 128.27 58.42)
 		)
 		(stroke
@@
 	(wire
 		(pts
-			(xy 124.46 58.42) (xy 133.35 58.42)
+			(xy 128.27 58.42) (xy 137.16 58.42)
 		)
 		(stroke
@@
 	(wire
 		(pts
-			(xy 124.46 49.53) (xy 124.46 50.8)
+			(xy 128.27 49.53) (xy 128.27 50.8)
 		)
 		(stroke
@@
 	(wire
 		(pts
-			(xy 124.46 50.8) (xy 133.35 50.8)
+			(xy 128.27 50.8) (xy 137.16 50.8)
 		)
 		(stroke
@@
 	(wire
 		(pts
-			(xy 115.57 50.8) (xy 124.46 50.8)
+			(xy 119.38 50.8) (xy 128.27 50.8)
 		)
 		(stroke
@@
 	(wire
 		(pts
-			(xy 124.46 62.23) (xy 121.92 62.23)
+			(xy 128.27 62.23) (xy 125.73 62.23)
 		)
 		(stroke
@@
 	(wire
 		(pts
-			(xy 148.59 62.23) (xy 124.46 62.23)
+			(xy 148.59 62.23) (xy 128.27 62.23)
 		)
 		(stroke
@@
 	(global_label "VM"
 		(shape input)
-		(at 121.92 62.23 180)
+		(at 125.73 62.23 180)
 		(fields_autoplaced yes)
 		(effects
@@
 		)
 		(property "Intersheetrefs" "${INTERSHEET_REFS}"
-			(at 117.5001 62.23 0)
+			(at 121.3101 62.23 0)
 			(effects
 				(font
@@
 	(symbol
 		(lib_id "Device:C")
-		(at 115.57 54.61 0)
+		(at 119.38 54.61 0)
 		(unit 1)
 		(exclude_from_sim no)
@@
 		(dnp no)
 		(property "Reference" "C7"
-			(at 117.856 53.594 0)
+			(at 121.666 53.594 0)
 			(effects
 				(font
@@
 		)
 		(property "Value" "10µF"
-			(at 117.856 56.134 0)
+			(at 121.666 56.134 0)
 			(effects
 				(font
@@
 		)
 		(property "Footprint" "Capacitor_SMD:C_1206_3216Metric"
-			(at 116.5352 58.42 0)
+			(at 120.3452 58.42 0)
 			(effects
 				(font
@@
 		)
 		(property "Datasheet" "~"
-			(at 115.57 54.61 0)
+			(at 119.38 54.61 0)
 			(effects
 				(font
@@
 		)
 		(property "Description" "Unpolarized capacitor"
-			(at 115.57 54.61 0)
+			(at 119.38 54.61 0)
 			(effects
 				(font
@@
 	(symbol
 		(lib_id "power:GND")
-		(at 124.46 49.53 180)
+		(at 128.27 49.53 180)
 		(unit 1)
 		(exclude_from_sim no)
@@
 		(fields_autoplaced yes)
 		(property "Reference" "#PWR07"
-			(at 124.46 43.18 0)
+			(at 128.27 43.18 0)
 			(effects
 				(font
@@
 		)
 		(property "Value" "GND"
-			(at 124.46 44.45 0)
+			(at 128.27 44.45 0)
 			(effects
 				(font
@@
 		)
 		(property "Footprint" ""
-			(at 124.46 49.53 0)
+			(at 128.27 49.53 0)
 			(effects
 				(font
@@
 		)
 		(property "Datasheet" ""
-			(at 124.46 49.53 0)
+			(at 128.27 49.53 0)
 			(effects
 				(font
@@
 		)
 		(property "Description" "Power symbol creates a global label with name \"GND\" , ground"
-			(at 124.46 49.53 0)
+			(at 128.27 49.53 0)
 			(effects
 				(font
@@
 	(symbol
 		(lib_id "Device:C")
-		(at 133.35 54.61 0)
+		(at 137.16 54.61 0)
 		(unit 1)
 		(exclude_from_sim no)
@@
 		(dnp no)
 		(property "Reference" "C6"
-			(at 135.89 53.34 0)
+			(at 139.7 53.34 0)
 			(effects
 				(font
@@
 		)
 		(property "Value" "10µF"
-			(at 135.89 55.88 0)
+			(at 139.7 55.88 0)
 			(effects
 				(font
@@
 		)
 		(property "Footprint" "Capacitor_SMD:C_1206_3216Metric"
-			(at 134.3152 58.42 0)
+			(at 138.1252 58.42 0)
 			(effects
 				(font
@@
 		)
 		(property "Datasheet" "~"
-			(at 133.35 54.61 0)
+			(at 137.16 54.61 0)
 			(effects
 				(font
@@
 		)
 		(property "Description" "Unpolarized capacitor"
-			(at 133.35 54.61 0)
+			(at 137.16 54.61 0)
 			(effects
 				(font
